Commit message: Add inertia values to urdf

File: lwr_description/model/kuka_lwr.urdf.xacro (robot description, xacro)
@@ -31,4 +31,5 @@
 				<mass value="${base_mass}"/>
 				<origin xyz="0 0 0.055"  />
+                <inertia ixx="0.00381666666667" ixy="0" ixz="0" iyy="0.0036" iyz="0" izz="0.00381666666667"/>
 				<cylinder_inertia_def radius="0.06" length="0.11" mass="${base_mass}"/>
 			</inertial>
@@ -68,4 +69,5 @@
 				<mass value="${link_mass}"/>
 				<origin rpy="0 0 0" xyz="0 -0.06 0.130"/>
+                <inertia ixx="0.0136666666667" ixy="0" ixz="0" iyy="0.003" iyz="0" izz="0.0118666666667"/>
 				<cuboid_inertia_def length="0.12" width="0.06" height="0.260" mass="${link_mass}"/>
 			</inertial>
@@ -117,4 +119,5 @@
 				<mass value="${link_mass}"/>
 				<origin rpy="0 0 0" xyz="0 0.06 ${0.130 - 0.06}"/>
+                <inertia ixx="0.0136666666667" ixy="0" ixz="0" iyy="0.003" iyz="0" izz="0.0118666666667"/>
 				<cuboid_inertia_def length="0.12" width="0.06" height="0.260" mass="${link_mass}"/>
 			</inertial>
@@ -166,4 +169,5 @@
 				<mass value="${link_mass}"/>
 				<origin rpy="0 0 0" xyz="0 0.06 0.130"/>
+                <inertia ixx="0.0136666666667" ixy="0" ixz="0" iyy="0.003" iyz="0" izz="0.0118666666667"/>
 				<cuboid_inertia_def length="0.12" width="0.06" height="0.260" mass="${link_mass}"/>
 			</inertial>
@@ -215,4 +219,5 @@
 				<mass value="${link_mass}"/>
 				<origin rpy="0 0 0" xyz="0 -0.06 ${0.130 - 0.06}"/>
+                <inertia ixx="0.0136666666667" ixy="0" ixz="0" iyy="0.003" iyz="0" izz="0.0118666666667"/>
 				<cuboid_inertia_def length="0.12" width="0.06" height="0.2600" mass="${link_mass}"/>
 			</inertial>
@@ -264,4 +269,5 @@
 				<mass value="${link_mass}"/>
 				<origin rpy="0 0 0" xyz="0 0 0.124"/>
+                <inertia ixx="0.0126506666667" ixy="0" ixz="0" iyy="0.003" iyz="0" izz="0.0108506666667"/>
 				<cuboid_inertia_def length="0.12" width="0.06" height="0.248" mass="${link_mass}"/>
 			</inertial>
@@ -313,4 +319,5 @@
 				<mass value="${wrist_mass}"/>
 				<origin rpy="0 0 0" xyz="0 0 0.0625"/>
+                <inertia ixx="0.000520833333333" ixy="0" ixz="0" iyy="0.000520833333333" iyz="0" izz="0.000520833333333"/>
 				<cuboid_inertia_def length="0.125" width="0.125" height="0.125" mass="${wrist_mass}"/>
 			</inertial>
@@ -350,4 +357,5 @@
 				<mass value="${tip_mass}"/>
 				<origin xyz="0 0 0"/>
+                <inertia ixx="0.0333333333333" ixy="0" ixz="0" iyy="0.0333333333333" iyz="0" izz="0.0333333333333"/>
 				<cuboid_inertia_def length="0.1" width="0.1" height="0.1" mass="${tip_mass}"/>
 			</inertial>
