Commit message: Change urdf to include ft sensor

File: lwr_description/model/kuka_lwr.gazebo.xacro (robot description, xacro)
@@ -9,29 +9,29 @@
 		<gazebo reference="${name}_base_link">
 			<gravity>true</gravity>
-			<material>Gazebo/Orange</material>
+			<material>Gazebo/Blue</material>
 		</gazebo>
 		<gazebo reference="${name}_1_link">
 			<gravity>true</gravity>
-			<material>Gazebo/Orange</material>
+			<material>Gazebo/Blue</material>
 		</gazebo>
 		<gazebo reference="${name}_2_link">
 			<gravity>true</gravity>
-			<material>Gazebo/Orange</material>
+			<material>Gazebo/Blue</material>
 		</gazebo>
 		<gazebo reference="${name}_3_link">
 			<gravity>true</gravity>
-			<material>Gazebo/Orange</material>
+			<material>Gazebo/Blue</material>
 		</gazebo>
 		<gazebo reference="${name}_4_link">
 			<gravity>true</gravity>
-			<material>Gazebo/Orange</material>
+			<material>Gazebo/Blue</material>
 		</gazebo>
 		<gazebo reference="${name}_5_link">
 			<gravity>true</gravity>
-			<material>Gazebo/Orange</material>
+			<material>Gazebo/Blue</material>
 		</gazebo>
 		<gazebo reference="${name}_6_link">
 			<gravity>true</gravity>
-			<material>Gazebo/Orange</material>
+			<material>Gazebo/Blue</material>
 		</gazebo>
 		<gazebo reference="${name}_7_link">
@@ -39,4 +39,20 @@
 			<material>Gazebo/Grey</material>
 		</gazebo>
+		<gazebo reference="adaptor_kuka">
+			<gravity>true</gravity>
+			<material>Gazebo/Grey</material>
+		</gazebo>
+		<gazebo reference="force_torque_sensor">
+			<gravity>true</gravity>
+			<material>Gazebo/White</material>
+		</gazebo>
+		<gazebo reference="end_effector">
+			<gravity>true</gravity>
+			<material>Gazebo/Grey</material>
+		</gazebo>
+		<gazebo reference="end_effector_sponge">
+			<gravity>true</gravity>
+			<material>Gazebo/White</material>
+		</gazebo>
 	</xacro:macro>
 </robot>

File: lwr_description/model/kuka_lwr.urdf.xacro (robot description, xacro)
@@ -365,6 +365,13 @@
 					<mesh filename="package://lwr_description/meshes/lwr4plus/visual/link_7.STL"/>
 				</geometry>
-			<material name="Kuka/DarkGrey"/>
-			</visual>
+                <material name="Kuka/DarkGrey"/>
+			</visual>
+            <visual>
+                <origin rpy="0 0 0" xyz="0 0 0.015"/>
+                <geometry>
+                    <cylinder radius="0.03" length="0.03"/>
+                </geometry>
+                <material name="Kuka/DarkGrey"/>
+            </visual>
 			<collision>
 			<origin xyz="0 0 0" rpy="0 0 ${M_PI}"/>
@@ -374,4 +381,94 @@
 			</collision>
 		</link>
+		<joint name="${name}_a7_joint" type="fixed">
+            <origin rpy="0 0 3.14159265359" xyz="0 0 0.03"/>
+			<parent link="${name}_7_link"/>
+			<child link="adaptor_kuka"/>
+		</joint>
+        <link name="adaptor_kuka">
+            <inertial>
+                <mass value="0.1"/>
+                <origin xyz="0 0 0"/>
+                <inertia ixx="0.01" ixy="0" ixz="0" iyy="0.01" iyz="0" izz="0.01"/>
+            </inertial>
+            <visual>
+                <origin rpy="0 0 0" xyz="0 0 0.0"/>
+                <geometry>
+                    <mesh filename="package://lwr_description/meshes/lwr4plus/visual/adaptor_kuka.stl" scale="0.001 0.001 0.001"/>
+                </geometry>
+                <material name="Kuka/DarkGrey"/>
+            </visual>
+        </link>
+            <!-- FORCE TORQUE SENSOR -->
+        <joint name="force_torque_sensor_mount" type="fixed">
+            <origin rpy="0 0 0" xyz="0 0 0.0453"/>
+            <parent link="adaptor_kuka"/>
+            <child link="force_torque_sensor"/>
+        </joint>
+        <link name="force_torque_sensor">
+            <inertial>
+                <mass value="0.5"/>
+                <origin xyz="-0.000007 0.001524 0.027591"/>
+                <inertia ixx="0.0333333333333" ixy="0" ixz="0" iyy="0.0333333333333" iyz="0" izz="0.0333333333333"/>
+            </inertial>
+            <visual>
+                <origin rpy="0 0 0" xyz="0 0 0"/>
+                <material name="Kuka/LightGrey"/>
+                <geometry>
+                    <mesh filename="package://lwr_description/meshes/lwr4plus/visual/force_sensor.stl" scale="0.001 0.001 0.001"/>
+                </geometry>
+            </visual>
+        </link>
+            <!-- END-EFFECTOR TOOL CONE -->
+        <joint name="end_effector_joint" type="fixed">
+            <origin rpy="0 0 0.0" xyz="0 0 0.020"/>
+            <parent link="force_torque_sensor"/>
+            <child link="end_effector"/>
+        </joint>
+        <link name="end_effector">
+            <inertial>
+                <mass value="1"/>
+                <origin xyz="-0.000007 0.001524 0.027591"/>
+                <inertia ixx="0.00409836" ixy="0.000000" ixz="0.000000" iyy="0.00061475" iyz="0.000000" izz="0.00409836"/>
+            </inertial>
+            <visual>
+                <origin rpy="0 0 0" xyz="0 0 0"/>
+                <material name="Kuka/DarkGrey"/>
+                <geometry>
+                    <mesh filename="package://lwr_description/meshes/lwr4plus/visual/adaptor_endeffector.stl" scale="0.001 0.001 0.001"/>
+                </geometry>
+            </visual>
+            <collision>
+                <geometry>
+                    <mesh filename="package://lwr_description/meshes/lwr4plus/visual/adaptor_endeffector.stl" scale="0.001 0.001 0.001"/>
+                </geometry>
+            </collision>
+        </link>
+            <!-- SPONGE AT THE END -->
+        <joint name="end_effector_joint_sponge" type="fixed">
+            <origin rpy="0 0 0.0" xyz="0 0 0.0026"/>
+            <parent link="end_effector"/>
+            <child link="end_effector_sponge"/>
+        </joint>
+        <link name="end_effector_sponge">
+            <inertial>
+                <mass value="1"/>
+                <origin xyz="-0.000007 0.001524 0.027591"/>
+                <inertia ixx="0.00409836" ixy="0.000000" ixz="0.000000" iyy="0.00061475" iyz="0.000000" izz="0.00409836"/>
+            </inertial>
+            <visual>
+                <origin rpy="0 0 0" xyz="0 0 0"/>
+                <geometry>
+                    <cylinder length="0.005" radius="0.04"/>
+                </geometry>
+                <material name="Kuka/Silver"/>
+            </visual>
+            <collision>
+                <origin rpy="0 0 0" xyz="0 0 0"/>
+                <geometry>
+                    <cylinder length="0.005" radius="0.04"/>
+                </geometry>
+            </collision>
+        </link>
 		<xacro:kuka_lwr_gazebo name="${name}"/>
 		<xacro:kuka_lwr_transmission name="${name}"/>
